Commit message: skid steer

File: urdf/robot.xacro (robot description, xacro)
@@ -26,5 +26,5 @@
           </geometry>
           <mass value="0.998"/>
-          <inertia ixx="0.098875000000000005" ixy="0" ixz="0" iyy="0.098875000000000005" iyz="0" izz="0.11300000000000002"/>
+          <inertia ixx="0.017465000000000001" ixy="0" ixz="0" iyy="0.017465000000000001" iyz="0" izz="0.019960000000000002"/>
       </inertial>
   </link>
@@ -34,4 +34,31 @@
       <child link="base_link"/>
   </joint>
+  <gazebo reference="base_link">
+      <selfCollide>true</selfCollide>
+      <mu1 value="200.0"/>
+      <mu2 value="100.0"/>
+      <kp value="10000000.0"/>
+      <kd value="1.0"/>
+  </gazebo>
+  <link name="fork_link">
+      <collision>
+          <origin rpy="0 0 0" xyz="0 0 0"/>
+          <geometry>
+              <box size="0.005 0.04 0.002"/>
+          </geometry>
+      </collision>
+  </link>
+  <joint name="fork_joint" type="fixed">
+      <origin xyz="0.031 0.0 0.005" rpy="0 0 0"/>
+      <parent link="base_link"/>
+      <child link="fork_link"/>
+  </joint>
+  <gazebo reference="fork_link">
+      <selfCollide>true</selfCollide>
+      <mu1 value="200.0"/>
+      <mu2 value="100.0"/>
+      <kp value="10000000.0"/>
+      <kd value="1.0"/>
+  </gazebo>
   <xacro:macro name="wheel" params="link_name pos_x pos_y pos_z">
     <link name="${link_name}">
@@ -51,5 +78,5 @@
         <parent link="base_link"/>
         <child link="${link_name}"/>
-          <origin rpy="${pi/2} 0 0" xyz="${pos_x} ${pos_y} ${pos_z}"/>
+          <origin rpy="${-pi/2} 0 0" xyz="${pos_x} ${pos_y} ${pos_z}"/>
         <axis xyz="0 0 1"/>
     </joint>
@@ -69,4 +96,5 @@
  <xacro:wheel link_name="front_right_wheel" pos_x=" 0.015" pos_y="-0.02" pos_z="0.01"/>
  <xacro:wheel link_name="front_left_wheel"  pos_x=" 0.015" pos_y=" 0.02" pos_z="0.01"/>
+ <!-- transmission -->
  <gazebo>
      <plugin name="skid_steer_drive_controller" filename="libgazebo_ros_skid_steer_drive.so">
@@ -90,3 +118,43 @@
      </plugin>
  </gazebo>
+ <!-- sensors -->
+ <link name="imu_link">
+     <visual>
+       <geometry>
+           <box size="0.001 0.001 0.001"/>
+       </geometry>
+     </visual>
+     <collision>
+       <geometry>
+         <box size="0.001 0.001 0.001"/>
+       </geometry>
+     </collision>
+     <inertial>
+         <mass value="0.008"/>
+         <inertia ixx="6.1066666666666663e-07" ixy="0" ixz="0" iyy="6.1066666666666663e-07" iyz="0" izz="1.1999999999999999e-06"/>
+     </inertial>
+ </link>
+ <joint name="imu_joint" type="fixed">
+     <parent link="base_link"/>
+     <child link="imu_link"/>
+     <origin rpy="0 0 0" xyz="0 0 0.05"/>
+ </joint>
+ <gazebo reference="imu_link">
+  <gravity>true</gravity>
+  <sensor name="imu_sensor" type="imu">
+    <always_on>true</always_on>
+    <update_rate>100</update_rate>
+    <visualize>true</visualize>
+    <topic>imu/data_raw</topic>
+    <plugin filename="libgazebo_ros_imu_sensor.so" name="imu_plugin">
+      <topicName>imu/data_raw</topicName>
+      <bodyName>imu_link</bodyName>
+      <updateRateHZ>100.0</updateRateHZ>
+      <gaussianNoise>0.0001</gaussianNoise>
+      <xyzOffset>0 0 0</xyzOffset>
+      <rpyOffset>0 3.14 0</rpyOffset>
+      <frameName>imu_link</frameName>
+    </plugin>
+  </sensor>
+ </gazebo>
 </robot>

Commit message: camera

File: urdf/robot.xacro (robot description, xacro)
@@ -119,4 +119,48 @@
  </gazebo>
  <!-- sensors -->
+  <link name="head_camera">
+    <visual>
+        <origin rpy="0 ${pi/2} 0" xyz="0 0 0"/>
+        <geometry>
+          <cylinder length="0.001" radius="0.002"/>
+        </geometry>
+    </visual>
+  </link>
+  <joint name="head_camera_joint" type="fixed">
+    <parent link="base_link"/>
+    <child link="head_camera"/>
+    <origin rpy="0 0 0" xyz="0.02 0 0.033"/>
+  </joint>
+  <gazebo reference="head_camera">
+  <sensor type="camera" name="head_camera">
+    <update_rate>30.0</update_rate>
+    <camera name="head_camera">
+      <horizontal_fov>2.0</horizontal_fov>
+      <image>
+        <width>1920</width>
+        <height>1080</height>
+        <format>R8G8B8</format>
+      </image>
+      <clip>
+        <near>0.01</near>
+        <far>100.0</far>
+      </clip>
+    </camera>
+    <plugin name="camera_controller" filename="libgazebo_ros_camera.so">
+      <alwaysOn>true</alwaysOn>
+      <updateRate>30.0</updateRate>
+      <cameraName>head_camera</cameraName>
+      <imageTopicName>image_raw</imageTopicName>
+      <cameraInfoTopicName>camera_info</cameraInfoTopicName>
+      <frameName>head_camera</frameName>
+      <hackBaseline>0.07</hackBaseline>
+      <distortionK1>0.0</distortionK1>
+      <distortionK2>0.0</distortionK2>
+      <distortionK3>0.0</distortionK3>
+      <distortionT1>0.0</distortionT1>
+      <distortionT2>0.0</distortionT2>
+    </plugin>
+  </sensor>
+  </gazebo>
  <link name="imu_link">
      <visual>
@@ -153,5 +197,5 @@
       <gaussianNoise>0.0001</gaussianNoise>
       <xyzOffset>0 0 0</xyzOffset>
-      <rpyOffset>0 3.14 0</rpyOffset>
+      <rpyOffset>0 0 0</rpyOffset>
       <frameName>imu_link</frameName>
     </plugin>

Commit message: cliff sensors

File: urdf/robot.xacro (robot description, xacro)
@@ -18,5 +18,5 @@
           <origin rpy="0.0 0 0" xyz="-0.009 0 0.02"/>
           <geometry>
-              <box size="0.06 0.025 0.035"/>
+              <box size="0.06 0.025 0.03"/>
           </geometry>
       </collision>
@@ -118,87 +118,7 @@
      </plugin>
  </gazebo>
- <!-- sensors -->
-  <link name="head_camera">
-    <visual>
-        <origin rpy="0 ${pi/2} 0" xyz="0 0 0"/>
-        <geometry>
-          <cylinder length="0.001" radius="0.002"/>
-        </geometry>
-    </visual>
-  </link>
-  <joint name="head_camera_joint" type="fixed">
-    <parent link="base_link"/>
-    <child link="head_camera"/>
-    <origin rpy="0 0 0" xyz="0.02 0 0.033"/>
-  </joint>
-  <gazebo reference="head_camera">
-  <sensor type="camera" name="head_camera">
-    <update_rate>30.0</update_rate>
-    <camera name="head_camera">
-      <horizontal_fov>2.0</horizontal_fov>
-      <image>
-        <width>1280</width>
-        <height>720</height>
-        <format>R8G8B8</format>
-      </image>
-      <clip>
-        <near>0.01</near>
-        <far>100.0</far>
-      </clip>
-    </camera>
-    <plugin name="camera_controller" filename="libgazebo_ros_camera.so">
-      <alwaysOn>true</alwaysOn>
-      <updateRate>30.0</updateRate>
-      <cameraName>head_camera</cameraName>
-      <imageTopicName>image_raw</imageTopicName>
-      <cameraInfoTopicName>camera_info</cameraInfoTopicName>
-      <frameName>head_camera</frameName>
-      <hackBaseline>0.07</hackBaseline>
-      <distortionK1>0.0</distortionK1>
-      <distortionK2>0.0</distortionK2>
-      <distortionK3>0.0</distortionK3>
-      <distortionT1>0.0</distortionT1>
-      <distortionT2>0.0</distortionT2>
-    </plugin>
-  </sensor>
-  </gazebo>
- <link name="imu_link">
-     <visual>
-       <geometry>
-           <box size="0.001 0.001 0.001"/>
-       </geometry>
-     </visual>
-     <collision>
-       <geometry>
-         <box size="0.001 0.001 0.001"/>
-       </geometry>
-     </collision>
-     <inertial>
-         <mass value="0.008"/>
-         <inertia ixx="6.1066666666666663e-07" ixy="0" ixz="0" iyy="6.1066666666666663e-07" iyz="0" izz="1.1999999999999999e-06"/>
-     </inertial>
- </link>
- <joint name="imu_joint" type="fixed">
-     <parent link="base_link"/>
-     <child link="imu_link"/>
-     <origin rpy="0 0 0" xyz="0 0 0.05"/>
- </joint>
- <gazebo reference="imu_link">
-  <gravity>true</gravity>
-  <sensor name="imu_sensor" type="imu">
-    <always_on>true</always_on>
-    <update_rate>100</update_rate>
-    <visualize>true</visualize>
-    <topic>imu/data_raw</topic>
-    <plugin filename="libgazebo_ros_imu_sensor.so" name="imu_plugin">
-      <topicName>imu/data_raw</topicName>
-      <bodyName>imu_link</bodyName>
-      <updateRateHZ>100.0</updateRateHZ>
-      <gaussianNoise>0.0001</gaussianNoise>
-      <xyzOffset>0 0 0</xyzOffset>
-      <rpyOffset>0 0 0</rpyOffset>
-      <frameName>imu_link</frameName>
-    </plugin>
-  </sensor>
- </gazebo>
+<!-- sensors -->
+<xacro:include filename="$(find vector_description)/urdf/cliff_sensor.xacro"/>
+<xacro:include filename="$(find vector_description)/urdf/imu.xacro"/>
+<xacro:include filename="$(find vector_description)/urdf/camera.xacro"/>
 </robot>

Commit message: tof sensor

File: urdf/robot.xacro (robot description, xacro)
@@ -18,5 +18,5 @@
           <origin rpy="0.0 0 0" xyz="-0.009 0 0.02"/>
           <geometry>
-              <box size="0.06 0.025 0.03"/>
+              <box size="0.055 0.025 0.03"/>
           </geometry>
       </collision>
@@ -122,3 +122,4 @@
 <xacro:include filename="$(find vector_description)/urdf/imu.xacro"/>
 <xacro:include filename="$(find vector_description)/urdf/camera.xacro"/>
+<xacro:include filename="$(find vector_description)/urdf/nir_tof.xacro"/>
 </robot>
