Commit message: changed topics to match driver

File: urdf/camera.xacro (robot description, xacro)
@@ -33,6 +33,6 @@
       <updateRate>30.0</updateRate>
       <cameraName>head_camera</cameraName>
-      <imageTopicName>image_raw</imageTopicName>
-      <cameraInfoTopicName>camera_info</cameraInfoTopicName>
+      <imageTopicName>/vector/camera</imageTopicName>
+      <cameraInfoTopicName>/vector/camera_info</cameraInfoTopicName>
       <frameName>head_camera</frameName>
       <hackBaseline>0.07</hackBaseline>

File: urdf/cliff_sensor.xacro (robot description, xacro)
@@ -2,5 +2,5 @@
 <robot xmlns:xacro="http://www.ros.org/wiki/xacro">
 <xacro:macro name="cliff" params="link_name pos_x pos_y pos_z">
-  <link name="${link_name}">
+  <link name="${link_name}_cliff">
       <visual>
           <geometry>
@@ -9,11 +9,11 @@
       </visual>
   </link>
-  <joint name="${link_name}_joint" type="fixed">
+  <joint name="${link_name}_cliff_joint" type="fixed">
       <parent link="base_link"/>
-      <child link="${link_name}"/>
+      <child link="${link_name}_cliff"/>
       <origin rpy="0 ${pi/2} 0" xyz="${pos_x} ${pos_y} ${pos_z}"/>
   </joint>
-  <gazebo reference="${link_name}">
-      <sensor type="ray" name="${link_name}">
+  <gazebo reference="${link_name}_cliff">
+      <sensor type="ray" name="${link_name}_cliff">
           <pose>0 0 0 0 0 0</pose>
           <visualize>false</visualize>
@@ -47,5 +47,5 @@
           <plugin filename="libgazebo_ros_range.so" name="gazebo_ros_range">
               <gaussianNoise>0.01</gaussianNoise>
-              <topicName>/cliff/${link_name}</topicName>
+              <topicName>/vector/cliff/${link_name}</topicName>
               <frameName>${link_name}</frameName>
               <radiation>INFRARED</radiation>

File: urdf/imu.xacro (robot description, xacro)
@@ -28,5 +28,5 @@
    <update_rate>100</update_rate>
    <visualize>true</visualize>
-   <topic>imu/data_raw</topic>
+   <topic>vector/imu</topic>
    <plugin filename="libgazebo_ros_imu_sensor.so" name="imu_plugin">
      <topicName>imu/data_raw</topicName>

File: urdf/nir_tof.xacro (robot description, xacro)
@@ -39,6 +39,6 @@
               </scan>
               <range>
-                  <min>0.01</min>
-                  <max>1.0</max>
+                  <min>0.0</min>
+                  <max>0.3</max>
                   <resolution>0.01</resolution>
               </range>
@@ -51,5 +51,5 @@
           <plugin filename="libgazebo_ros_range.so" name="gazebo_ros_range">
               <gaussianNoise>0.01</gaussianNoise>
-              <topicName>/tof</topicName>
+              <topicName>/vector/laser</topicName>
               <frameName>tof_link</frameName>
               <radiation>INFRARED</radiation>

Commit message: incorporating construct model

File: urdf/camera.xacro (robot description, xacro)
@@ -1,47 +1,46 @@
 <?xml version="1.0"?>
 <robot xmlns:xacro="http://www.ros.org/wiki/xacro">
-  <link name="head_camera">
-    <visual>
-        <origin rpy="0 ${pi/2} 0" xyz="0 0 0"/>
-        <geometry>
-          <cylinder length="0.001" radius="0.002"/>
-        </geometry>
-    </visual>
-  </link>
+    <link name="camera_link">
+    </link>
   <joint name="head_camera_joint" type="fixed">
-    <parent link="base_link"/>
-    <child link="head_camera"/>
-    <origin rpy="0 0 0" xyz="0.02 0 0.033"/>
+    <parent link="head"/>
+    <child link="camera_link"/>
+    <origin xyz="0.020813 0 -0.0071471" rpy="0 0 0"/>
   </joint>
-  <gazebo reference="head_camera">
-  <sensor type="camera" name="head_camera">
-    <update_rate>30.0</update_rate>
-    <camera name="head_camera">
-      <horizontal_fov>2.0</horizontal_fov>
-      <image>
-        <width>1280</width>
-        <height>720</height>
-        <format>R8G8B8</format>
-      </image>
-      <clip>
-        <near>0.01</near>
-        <far>100.0</far>
-      </clip>
-    </camera>
-    <plugin name="camera_controller" filename="libgazebo_ros_camera.so">
-      <alwaysOn>true</alwaysOn>
-      <updateRate>30.0</updateRate>
-      <cameraName>head_camera</cameraName>
-      <imageTopicName>/vector/camera</imageTopicName>
-      <cameraInfoTopicName>/vector/camera_info</cameraInfoTopicName>
-      <frameName>head_camera</frameName>
-      <hackBaseline>0.07</hackBaseline>
-      <distortionK1>0.0</distortionK1>
-      <distortionK2>0.0</distortionK2>
-      <distortionK3>0.0</distortionK3>
-      <distortionT1>0.0</distortionT1>
-      <distortionT2>0.0</distortionT2>
-    </plugin>
-  </sensor>
+  <gazebo reference="camera_link">
+    <sensor type="camera" name="cozmo_camera">
+      <update_rate>10.0</update_rate>
+      <camera name="headcamera">
+        <horizontal_fov>1.3962634</horizontal_fov>
+        <image>
+          <width>1280</width>
+          <height>720</height>
+          <format>R8G8B8</format>
+        </image>
+        <clip>
+          <near>0.01</near>
+          <far>100</far>
+        </clip>
+        <noise>
+          <type>gaussian</type>
+          <mean>0.0</mean>
+          <stddev>0.007</stddev>
+        </noise>
+      </camera>
+      <plugin name="camera_controller" filename="libgazebo_ros_camera.so">
+        <alwaysOn>true</alwaysOn>
+        <updateRate>25.0</updateRate>
+        <cameraName>camera</cameraName>
+        <imageTopicName>image</imageTopicName>
+        <cameraInfoTopicName>camera_info</cameraInfoTopicName>
+        <frameName>camera_link</frameName>
+        <hackBaseline>0.07</hackBaseline>
+        <distortionK1>0.0</distortionK1>
+        <distortionK2>0.0</distortionK2>
+        <distortionK3>0.0</distortionK3>
+        <distortionT1>0.0</distortionT1>
+        <distortionT2>0.0</distortionT2>
+      </plugin>
+    </sensor>
   </gazebo>
 </robot>

File: urdf/imu.xacro (robot description, xacro)
@@ -1,42 +1,29 @@
 <?xml version="1.0"?>
 <robot xmlns:xacro="http://www.ros.org/wiki/xacro">
-<link name="imu_link">
-    <visual>
-      <geometry>
-          <box size="0.001 0.001 0.001"/>
-      </geometry>
-    </visual>
-    <collision>
-      <geometry>
-        <box size="0.001 0.001 0.001"/>
-      </geometry>
-    </collision>
-    <inertial>
-        <mass value="0.008"/>
-        <inertia ixx="6.1066666666666663e-07" ixy="0" ixz="0" iyy="6.1066666666666663e-07" iyz="0" izz="1.1999999999999999e-06"/>
-    </inertial>
-</link>
-<joint name="imu_joint" type="fixed">
-    <parent link="base_link"/>
-    <child link="imu_link"/>
-    <origin rpy="0 0 0" xyz="0 0 0.05"/>
-</joint>
-<gazebo reference="imu_link">
- <gravity>true</gravity>
- <sensor name="imu_sensor" type="imu">
-   <always_on>true</always_on>
-   <update_rate>100</update_rate>
-   <visualize>true</visualize>
-   <topic>vector/imu</topic>
-   <plugin filename="libgazebo_ros_imu_sensor.so" name="imu_plugin">
-     <topicName>imu/data_raw</topicName>
-     <bodyName>imu_link</bodyName>
-     <updateRateHZ>100.0</updateRateHZ>
-     <gaussianNoise>0.0001</gaussianNoise>
-     <xyzOffset>0 0 0</xyzOffset>
-     <rpyOffset>0 0 0</rpyOffset>
-     <frameName>imu_link</frameName>
-   </plugin>
- </sensor>
-</gazebo>
+    <link name="imu">
+    </link>
+  <joint name="imu_joint" type="fixed">
+    <parent link="head"/>
+    <child link="imu"/>
+    <origin xyz="0.0 0 0.0" rpy="0 0 0" />
+  </joint>
+  <gazebo reference="imu">
+    <gravity>true</gravity>
+    <sensor name="imu_sensor" type="imu">
+      <always_on>true</always_on>
+      <update_rate>100</update_rate>
+      <visualize>true</visualize>
+      <topic>__default_topic__</topic>
+      <plugin filename="libgazebo_ros_imu_sensor.so" name="imu_plugin">
+        <topicName>imu</topicName>
+        <bodyName>imu</bodyName>
+        <updateRateHZ>10.0</updateRateHZ>
+        <gaussianNoise>${0.0017*0.0017}</gaussianNoise>
+        <xyzOffset>0 0 0</xyzOffset>
+        <rpyOffset>0 0 0</rpyOffset>
+        <frameName>imu</frameName>
+      </plugin>
+      <pose>0 0 0 0 0 0</pose>
+    </sensor>
+  </gazebo>
 </robot>
