Commit message: fix the position of tof and tof frame rate
decrease the frame rate to be just lije the real one 
the position of the tof is wrong and it had false measurment

File: urdf/laser.xacro (robot description, xacro)
@@ -6,5 +6,5 @@
       <parent link="base_link"/>
       <child link="tof_link"/>
-      <origin rpy="0 0 0" xyz="0.042 0 -0.005"/>
+      <origin rpy="0 0 0" xyz="0.043 0 -0.005"/>
   </joint>
   <gazebo reference="tof_link">
@@ -12,5 +12,5 @@
           <pose>0 0 0 0 0 0</pose>
           <visualize>true</visualize>
-          <update_rate>20.0</update_rate>
+          <update_rate>10.0</update_rate>
           <ray>
               <scan>
@@ -44,5 +44,5 @@
               <frameName>tof_link</frameName>
               <radiation>INFRARED</radiation>
-              <updateRate>20</updateRate>
+              <updateRate>10</updateRate>
               <fov>${field_of_view}</fov>
           </plugin>
