Commit message: cozmo vs. vector

File: urdf/cozmo.xacro (robot description, xacro)
@@ -1,5 +1,5 @@
 <?xml version="1.0"?>
 <robot name="cozmo" xmlns:xacro="http://www.ros.org/wiki/xacro">
-  <xacro:include filename="$(find anki_description)/urdf/base.xacro"/>
+  <!-- Inertia util -->
   <xacro:include filename="$(find anki_description)/urdf/inertia.xacro"/>
   <link name="base_footprint"/>
@@ -9,8 +9,10 @@
     <child link="base_link"/>
   </joint>
+  <!-- Body -->
   <link name="base_link">
     <xacro:box_inertial mass="0.06" x="0.073" y="0.043" z="0.061" />
     <visual>
       <geometry>
+        <!-- TODO: check why this collada file won't load into gazebo -->
         <mesh filename="package://cozmo_description/meshes/body3.dae"  />
       </geometry>
@@ -22,4 +24,11 @@
     </collision>
   </link>
+  <gazebo reference="base_link">
+      <selfCollide>true</selfCollide>
+      <mu1 value="200.0"/>
+      <mu2 value="100.0"/>
+      <kp value="10000000.0"/>
+      <kd value="1.0"/>
+  </gazebo>
   <!-- Head -->
   <link name="head">
@@ -36,4 +45,11 @@
     </collision>
   </link>
+  <gazebo reference="head">
+      <kp>1000000000.0</kp>
+      <kd>1000000000.0</kd>
+      <mu1>10.0</mu1>
+      <mu2>10.0</mu2>
+      <self_collide>0</self_collide>
+  </gazebo>
   <!-- lifter -->
   <link name="full_lift">
@@ -50,220 +66,9 @@
     </collision>
   </link>
-  <!-- sensors links -->
-  <link name="camera_link">
-    <visual>
-      <geometry>
-        <box size="0.005 0.005 0.005"/>
-      </geometry>
-    </visual>
-  </link>
-  <link name="drop_ir">
-    <visual>
-      <geometry>
-        <box size="0.005 0.005 0.005"/>
-      </geometry>
-    </visual>
-  </link>
-  <link name="imu">
-    <visual>
-      <geometry>
-        <box size="0.005 0.005 0.005"/>
-      </geometry>
-    </visual>
-  </link>
-  <!-- JOINTS ====================================-->
-  <joint name="base_to_head" type="revolute">
-    <parent link="base_link"/>
-    <child link="head"/>
-    <origin xyz="0.0174507 0 0.022003"/>
-    <limit lower="-0.52" upper="0.17" effort="100" velocity="10"/>
-    <!-- Dampning break the model, keep it 0.0 -->
-    <dynamics damping="0.0" friction="0.1"/>
-    <axis xyz="0 1 0"/>
-  </joint>
-  <joint name="base_to_lift" type="revolute">
-    <parent link="base_link"/>
-    <child link="full_lift"/>
-    <origin xyz="-0.005 0 0.013"/>
-    <limit lower="-0.8" upper="0" effort="5" velocity="10"/>
-    <dynamics damping="0.0" friction="0.1"/>
-    <axis xyz="0 1 0"/>
-  </joint>
-  <joint name="head_camera_joint" type="fixed">
-    <parent link="head"/>
-    <child link="camera_link"/>
-    <origin xyz="0.020813 0 -0.0071471" rpy="0 0 0"/>
-  </joint>
-  <joint name="drop_ir_joint" type="fixed">
-    <parent link="base_link"/>
-    <child link="drop_ir"/>
-    <origin xyz="0.0351028 0 -0.0213898" rpy="0 1.57 0" />
-  </joint>
-  <joint name="imu_joint" type="fixed">
-    <parent link="head"/>
-    <child link="imu"/>
-    <origin xyz="0.0 0 0.0" rpy="0 0 0" />
-  </joint>
-  <gazebo reference="rear_right_wheel">
-    <mu1>0.5</mu1>
-    <mu2>0.5</mu2>
-  </gazebo>
-  <gazebo reference="rear_left_wheel">
-    <mu1>0.5</mu1>
-    <mu2>0.5</mu2>
-  </gazebo>
-<gazebo reference="front_right_wheel">
-    <mu1>100000</mu1>
-    <mu2>100000</mu2>
-  </gazebo>
-  <gazebo reference="front_left_wheel">
-    <mu1>100000</mu1>
-    <mu2>100000</mu2>
-  </gazebo>
-  <gazebo reference="head">
-      <kp>1000000000.0</kp>
-      <kd>1000000000.0</kd>
-      <mu1>10.0</mu1>
-      <mu2>10.0</mu2>
-      <self_collide>0</self_collide>
-  </gazebo>
-  <!-- Transmissions for joints -->
-  <transmission name="base_to_head_trans">
-      <type>transmission_interface/SimpleTransmission</type>
-      <joint name="base_to_head">
-        <hardwareInterface>hardware_interface/EffortJointInterface</hardwareInterface>
-      </joint>
-      <actuator name="base_to_headMotor">
-        <hardwareInterface>hardware_interface/EffortJointInterface</hardwareInterface>
-        <mechanicalReduction>1</mechanicalReduction>
-      </actuator>
-  </transmission>
-  <transmission name="base_to_lift_trans">
-      <type>transmission_interface/SimpleTransmission</type>
-      <joint name="base_to_lift">
-        <hardwareInterface>hardware_interface/EffortJointInterface</hardwareInterface>
-      </joint>
-      <actuator name="base_to_liftMotor">
-        <hardwareInterface>hardware_interface/EffortJointInterface</hardwareInterface>
-        <mechanicalReduction>1</mechanicalReduction>
-      </actuator>
-  </transmission>
-  <!-- ROS Control plugin for Gazebo -->
-  <gazebo>
-    <plugin name="gazebo_ros_control" filename="libgazebo_ros_control.so">
-      <robotNamespace>/cozmo</robotNamespace>
-      <legacyModeNS>true</legacyModeNS>
-    </plugin>
-  </gazebo>
-  <gazebo>
-  <plugin name="skid_steer_drive_controller" filename="libgazebo_ros_skid_steer_drive.so">
-    <updateRate>25.0</updateRate>
-    <robotNamespace>/</robotNamespace>
-    <leftFrontJoint>base_to_flw</leftFrontJoint>
-    <rightFrontJoint>base_to_frw</rightFrontJoint>
-    <leftRearJoint>base_to_rlw</leftRearJoint>
-    <rightRearJoint>base_to_rrw</rightRearJoint>
-    <wheelSeparation>0.048</wheelSeparation>
-    <wheelDiameter>0.026281</wheelDiameter>
-    <robotBaseFrame>base_link</robotBaseFrame>
-    <torque>20</torque>
-    <topicName>cmd_vel</topicName>
-    <commandTopic>cmd_vel</commandTopic>
-    <odometryTopic>odom</odometryTopic>
-    <odometryFrame>odom</odometryFrame>
-    <broadcastTF>1</broadcastTF>
-  </plugin>
-  </gazebo>
-  <gazebo reference="camera_link">
-    <sensor type="camera" name="cozmo_camera">
-      <update_rate>10.0</update_rate>
-      <camera name="headcamera">
-        <horizontal_fov>1.3962634</horizontal_fov>
-        <image>
-          <width>400</width>
-          <height>400</height>
-          <format>R8G8B8</format>
-        </image>
-        <clip>
-          <near>0.01</near>
-          <far>100</far>
-        </clip>
-        <noise>
-          <type>gaussian</type>
-          <mean>0.0</mean>
-          <stddev>0.007</stddev>
-        </noise>
-      </camera>
-      <plugin name="camera_controller" filename="libgazebo_ros_camera.so">
-        <alwaysOn>true</alwaysOn>
-        <updateRate>10.0</updateRate>
-        <cameraName>cozmo_camera</cameraName>
-        <imageTopicName>image</imageTopicName>
-        <cameraInfoTopicName>camera_info</cameraInfoTopicName>
-        <frameName>camera_link</frameName>
-        <hackBaseline>0.07</hackBaseline>
-        <distortionK1>0.0</distortionK1>
-        <distortionK2>0.0</distortionK2>
-        <distortionK3>0.0</distortionK3>
-        <distortionT1>0.0</distortionT1>
-        <distortionT2>0.0</distortionT2>
-      </plugin>
-    </sensor>
-  </gazebo>
-<gazebo reference="drop_ir">
- <sensor type="ray" name="TeraRanger">
-    <pose>0 0 0 0 0 0</pose>
-    <visualize>true</visualize>
-    <update_rate>50</update_rate>
-    <ray>
-       <scan>
-          <horizontal>
-             <samples>10</samples>
-             <resolution>1</resolution>
-             <min_angle>-0.14835</min_angle>
-             <max_angle>0.14835</max_angle>
-          </horizontal>
-          <vertical>
-             <samples>10</samples>
-             <resolution>1</resolution>
-             <min_angle>-0.14835</min_angle>
-             <max_angle>0.14835</max_angle>
-          </vertical>
-       </scan>
-       <range>
-          <min>0.01</min>
-          <max>2</max>
-          <resolution>0.02</resolution>
-       </range>
-    </ray>
-    <plugin filename="libgazebo_ros_range.so" name="gazebo_ros_range">
-       <gaussianNoise>0.005</gaussianNoise>
-       <alwaysOn>true</alwaysOn>
-       <updateRate>50</updateRate>
-       <topicName>drop_sensor</topicName>
-       <frameName>drop_ir</frameName>
-       <radiation>INFRARED</radiation>
-       <fov>0.2967</fov>
-    </plugin>
- </sensor>
- </gazebo>
-  <gazebo reference="imu">
-    <gravity>true</gravity>
-    <sensor name="imu_sensor" type="imu">
-      <always_on>true</always_on>
-      <update_rate>100</update_rate>
-      <visualize>true</visualize>
-      <topic>__default_topic__</topic>
-      <plugin filename="libgazebo_ros_imu_sensor.so" name="imu_plugin">
-        <topicName>imu</topicName>
-        <bodyName>imu</bodyName>
-        <updateRateHZ>10.0</updateRateHZ>
-        <gaussianNoise>${0.0017*0.0017}</gaussianNoise>
-        <xyzOffset>0 0 0</xyzOffset>
-        <rpyOffset>0 0 0</rpyOffset>
-        <frameName>imu</frameName>
-      </plugin>
-      <pose>0 0 0 0 0 0</pose>
-    </sensor>
-  </gazebo>
+  <!-- components -->
+  <xacro:include filename="$(find anki_description)/urdf/joints.xacro"/>
+  <xacro:include filename="$(find anki_description)/urdf/base.xacro"/>
+  <xacro:include filename="$(find anki_description)/urdf/cozmo_cam.xacro"/>
+  <xacro:include filename="$(find anki_description)/urdf/cozmo_drop.xacro"/>
+  <xacro:include filename="$(find anki_description)/urdf/imu.xacro"/>
 </robot>

File: urdf/imu.xacro (robot description, xacro)
@@ -1,6 +1,5 @@
 <?xml version="1.0"?>
 <robot xmlns:xacro="http://www.ros.org/wiki/xacro">
-    <link name="imu">
-    </link>
+  <link name="imu"/>
   <joint name="imu_joint" type="fixed">
     <parent link="head"/>

File: urdf/joints.xacro (robot description, xacro)
@@ -1,5 +1,4 @@
 <?xml version="1.0"?>
 <robot xmlns:xacro="http://www.ros.org/wiki/xacro">
-  <!-- JOINTS ====================================-->
   <joint name="base_to_head" type="revolute">
     <parent link="base_link"/>
@@ -7,5 +6,5 @@
     <origin xyz="0.0174507 0 0.022003"/>
     <limit lower="-0.52" upper="0.17" effort="100" velocity="10"/>
-    <!-- Dampning break the model, keep it 0.0 -->
+    <!-- Dampnening breaks the model (?), keep it 0.0 -->
     <dynamics damping="0.0" friction="0.1"/>
     <axis xyz="0 1 0"/>
@@ -19,11 +18,4 @@
     <axis xyz="0 1 0"/>
   </joint>
-  <gazebo reference="head">
-      <kp>1000000000.0</kp>
-      <kd>1000000000.0</kd>
-      <mu1>10.0</mu1>
-      <mu2>10.0</mu2>
-      <self_collide>0</self_collide>
-  </gazebo>
   <!-- Transmissions for joints -->
   <transmission name="base_to_head_trans">

File: urdf/vector.xacro (robot description, xacro)
@@ -44,4 +44,11 @@
     </collision>
   </link>
+  <gazebo reference="head">
+      <kp>1000000000.0</kp>
+      <kd>1000000000.0</kd>
+      <mu1>10.0</mu1>
+      <mu2>10.0</mu2>
+      <self_collide>0</self_collide>
+  </gazebo>
   <!-- lifter -->
   <link name="full_lift">
@@ -58,6 +65,10 @@
     </collision>
   </link>
-  <!-- Simulation -->
+  <!-- components -->
   <xacro:include filename="$(find anki_description)/urdf/joints.xacro"/>
   <xacro:include filename="$(find anki_description)/urdf/base.xacro"/>
+  <xacro:include filename="$(find anki_description)/urdf/vector_cam.xacro"/>
+  <xacro:include filename="$(find anki_description)/urdf/vector_drop.xacro"/>
+  <xacro:include filename="$(find anki_description)/urdf/imu.xacro"/>
+  <xacro:include filename="$(find anki_description)/urdf/laser.xacro"/>
 </robot>

File: urdf/vector_cam.xacro (robot description, xacro)
@@ -1,6 +1,5 @@
 <?xml version="1.0"?>
 <robot xmlns:xacro="http://www.ros.org/wiki/xacro">
-    <link name="camera_link">
-    </link>
+  <link name="camera_link"/>
   <joint name="head_camera_joint" type="fixed">
     <parent link="head"/>
@@ -9,5 +8,5 @@
   </joint>
   <gazebo reference="camera_link">
-    <sensor type="camera" name="cozmo_camera">
+    <sensor type="camera" name="vector_camera">
       <update_rate>10.0</update_rate>
       <camera name="headcamera">

Commit message: topic ns

File: urdf/cozmo.xacro (robot description, xacro)
@@ -72,3 +72,4 @@
   <xacro:include filename="$(find anki_description)/urdf/cozmo_drop.xacro"/>
   <xacro:include filename="$(find anki_description)/urdf/imu.xacro"/>
+  <xacro:imu name="cozmo"/>
 </robot>

File: urdf/cozmo_cam.xacro (robot description, xacro)
@@ -37,6 +37,6 @@
           <updateRate>10.0</updateRate>
           <cameraName>cozmo_camera</cameraName>
-          <imageTopicName>image</imageTopicName>
-          <cameraInfoTopicName>camera_info</cameraInfoTopicName>
+          <imageTopicName>/cozmo/image</imageTopicName>
+          <cameraInfoTopicName>/cozmo/camera_info</cameraInfoTopicName>
           <frameName>camera_link</frameName>
           <hackBaseline>0.07</hackBaseline>

File: urdf/cozmo_drop.xacro (robot description, xacro)
@@ -34,6 +34,6 @@
        </scan>
        <range>
-          <min>0.01</min>
-          <max>2</max>
+          <min>0.001</min>
+          <max>0.02</max>
           <resolution>0.02</resolution>
        </range>
@@ -43,5 +43,5 @@
        <alwaysOn>true</alwaysOn>
        <updateRate>50</updateRate>
-       <topicName>drop_sensor</topicName>
+       <topicName>/cozmo/drop_sensor</topicName>
        <frameName>drop_ir</frameName>
        <radiation>INFRARED</radiation>

File: urdf/imu.xacro (robot description, xacro)
@@ -1,4 +1,5 @@
 <?xml version="1.0"?>
 <robot xmlns:xacro="http://www.ros.org/wiki/xacro">
+<xacro:macro name="imu" params="ankirobot">
   <link name="imu"/>
   <joint name="imu_joint" type="fixed">
@@ -13,7 +14,7 @@
       <update_rate>100</update_rate>
       <visualize>true</visualize>
-      <topic>__default_topic__</topic>
+      <topic>${ankirobot}/imu</topic>
       <plugin filename="libgazebo_ros_imu_sensor.so" name="imu_plugin">
-        <topicName>imu</topicName>
+        <topicName>${ankirobot}/imu</topicName>
         <bodyName>imu</bodyName>
         <updateRateHZ>10.0</updateRateHZ>
@@ -26,3 +27,4 @@
     </sensor>
   </gazebo>
+</xacro:macro>
 </robot>

File: urdf/vector.xacro (robot description, xacro)
@@ -70,5 +70,6 @@
   <xacro:include filename="$(find anki_description)/urdf/vector_cam.xacro"/>
   <xacro:include filename="$(find anki_description)/urdf/vector_drop.xacro"/>
+  <xacro:include filename="$(find anki_description)/urdf/laser.xacro"/>
   <xacro:include filename="$(find anki_description)/urdf/imu.xacro"/>
-  <xacro:include filename="$(find anki_description)/urdf/laser.xacro"/>
+  <xacro:imu ankirobot="vector"/>
 </robot>

File: urdf/vector_cam.xacro (robot description, xacro)
@@ -29,8 +29,8 @@
       <plugin name="camera_controller" filename="libgazebo_ros_camera.so">
         <alwaysOn>true</alwaysOn>
-        <updateRate>25.0</updateRate>
+        <updateRate>10.0</updateRate>
         <cameraName>camera</cameraName>
-        <imageTopicName>image</imageTopicName>
-        <cameraInfoTopicName>camera_info</cameraInfoTopicName>
+        <imageTopicName>/vector/image</imageTopicName>
+        <cameraInfoTopicName>/vector/camera_info</cameraInfoTopicName>
         <frameName>camera_link</frameName>
         <hackBaseline>0.07</hackBaseline>

File: urdf/vector_drop.xacro (robot description, xacro)
@@ -1,179 +1,60 @@
 <?xml version="1.0"?>
 <robot xmlns:xacro="http://www.ros.org/wiki/xacro">
-    <link name="drop_ir_fl">
-    </link>
-    <link name="drop_ir_fr">
-    </link>
-    <link name="drop_ir_rl">
-    </link>
-    <link name="drop_ir_rr">
-    </link>
-  <joint name="drop_ir_fl_joint" type="fixed">
-    <parent link="base_link"/>
-    <child link="drop_ir_fl"/>
+  <xacro:macro name="drop_sensor" params="link_name *origin">
+    <link name="${link_name}"/>
+    <joint name="${link_name}_joint" type="fixed">
+        <parent link="base_link"/>
+        <child link="${link_name}"/>
+        <xacro:insert_block name="origin"/>
+    </joint>
+    <gazebo reference="${link_name}">
+     <sensor type="ray" name="ranger">
+        <pose>0 0 0 0 0 0</pose>
+        <visualize>true</visualize>
+        <update_rate>50</update_rate>
+        <ray>
+           <scan>
+              <horizontal>
+                 <samples>10</samples>
+                 <resolution>1</resolution>
+                 <min_angle>-0.14835</min_angle>
+                 <max_angle>0.14835</max_angle>
+              </horizontal>
+              <vertical>
+                 <samples>10</samples>
+                 <resolution>1</resolution>
+                 <min_angle>-0.14835</min_angle>
+                 <max_angle>0.14835</max_angle>
+              </vertical>
+           </scan>
+           <range>
+              <min>0.001</min>
+              <max>0.02</max>
+              <resolution>0.02</resolution>
+           </range>
+        </ray>
+        <plugin filename="libgazebo_ros_range.so" name="gazebo_ros_range">
+           <gaussianNoise>0.005</gaussianNoise>
+           <alwaysOn>true</alwaysOn>
+           <updateRate>50</updateRate>
+           <topicName>/vector/${link_name}</topicName>
+           <frameName>${link_name}</frameName>
+           <radiation>INFRARED</radiation>
+           <fov>0.2967</fov>
+        </plugin>
+     </sensor>
+     </gazebo>
+  </xacro:macro>
+  <xacro:drop_sensor link_name="drop_fl">
     <origin xyz="0.0351028 0.01 -0.0213898" rpy="0 1.57 0" />
-  </joint>
-  <joint name="drop_ir_fr_joint" type="fixed">
-    <parent link="base_link"/>
-    <child link="drop_ir_fr"/>
+  </xacro:drop_sensor>
+  <xacro:drop_sensor link_name="drop_fr">
     <origin xyz="0.0351028 -0.01 -0.0213898" rpy="0 1.57 0" />
-  </joint>
-  <joint name="drop_ir_rl_joint" type="fixed">
-    <parent link="base_link"/>
-    <child link="drop_ir_rl"/>
+  </xacro:drop_sensor>
+  <xacro:drop_sensor link_name="drop_rl">
     <origin xyz="-0.02 0.01 -0.0213898" rpy="0 1.57 0" />
-  </joint>
-  <joint name="drop_ir_rr_joint" type="fixed">
-    <parent link="base_link"/>
-    <child link="drop_ir_rr"/>
+  </xacro:drop_sensor>
+  <xacro:drop_sensor link_name="drop_rr">
     <origin xyz="-0.02 -0.01 -0.0213898" rpy="0 1.57 0" />
-  </joint>
-  <gazebo reference="drop_ir_fl">
-   <sensor type="ray" name="TeraRanger">
-      <pose>0 0 0 0 0 0</pose>
-      <visualize>true</visualize>
-      <update_rate>50</update_rate>
-      <ray>
-         <scan>
-            <horizontal>
-               <samples>10</samples>
-               <resolution>1</resolution>
-               <min_angle>-0.14835</min_angle>
-               <max_angle>0.14835</max_angle>
-            </horizontal>
-            <vertical>
-               <samples>10</samples>
-               <resolution>1</resolution>
-               <min_angle>-0.14835</min_angle>
-               <max_angle>0.14835</max_angle>
-            </vertical>
-         </scan>
-         <range>
-            <min>0.01</min>
-            <max>2</max>
-            <resolution>0.02</resolution>
-         </range>
-      </ray>
-      <plugin filename="libgazebo_ros_range.so" name="gazebo_ros_range">
-         <gaussianNoise>0.005</gaussianNoise>
-         <alwaysOn>true</alwaysOn>
-         <updateRate>50</updateRate>
-         <topicName>drop_sensor_fl</topicName>
-         <frameName>drop_ir_fl</frameName>
-         <radiation>INFRARED</radiation>
-         <fov>0.2967</fov>
-      </plugin>
-   </sensor>
-   </gazebo>
-  <gazebo reference="drop_ir_fr">
-   <sensor type="ray" name="TeraRanger">
-      <pose>0 0 0 0 0 0</pose>
-      <visualize>true</visualize>
-      <update_rate>50</update_rate>
-      <ray>
-         <scan>
-            <horizontal>
-               <samples>10</samples>
-               <resolution>1</resolution>
-               <min_angle>-0.14835</min_angle>
-               <max_angle>0.14835</max_angle>
-            </horizontal>
-            <vertical>
-               <samples>10</samples>
-               <resolution>1</resolution>
-               <min_angle>-0.14835</min_angle>
-               <max_angle>0.14835</max_angle>
-            </vertical>
-         </scan>
-         <range>
-            <min>0.01</min>
-            <max>2</max>
-            <resolution>0.02</resolution>
-         </range>
-      </ray>
-      <plugin filename="libgazebo_ros_range.so" name="gazebo_ros_range">
-         <gaussianNoise>0.005</gaussianNoise>
-         <alwaysOn>true</alwaysOn>
-         <updateRate>50</updateRate>
-         <topicName>drop_sensor_fr</topicName>
-         <frameName>drop_ir_fr</frameName>
-         <radiation>INFRARED</radiation>
-         <fov>0.2967</fov>
-      </plugin>
-   </sensor>
-   </gazebo>
-  <gazebo reference="drop_ir_rl">
-   <sensor type="ray" name="TeraRanger">
-      <pose>0 0 0 0 0 0</pose>
-      <visualize>true</visualize>
-      <update_rate>50</update_rate>
-      <ray>
-         <scan>
-            <horizontal>
-               <samples>10</samples>
-               <resolution>1</resolution>
-               <min_angle>-0.14835</min_angle>
-               <max_angle>0.14835</max_angle>
-            </horizontal>
-            <vertical>
-               <samples>10</samples>
-               <resolution>1</resolution>
-               <min_angle>-0.14835</min_angle>
-               <max_angle>0.14835</max_angle>
-            </vertical>
-         </scan>
-         <range>
-            <min>0.01</min>
-            <max>2</max>
-            <resolution>0.02</resolution>
-         </range>
-      </ray>
-      <plugin filename="libgazebo_ros_range.so" name="gazebo_ros_range">
-         <gaussianNoise>0.005</gaussianNoise>
-         <alwaysOn>true</alwaysOn>
-         <updateRate>50</updateRate>
-         <topicName>drop_sensor_rl</topicName>
-         <frameName>drop_ir_rl</frameName>
-         <radiation>INFRARED</radiation>
-         <fov>0.2967</fov>
-      </plugin>
-   </sensor>
-   </gazebo>
-  <gazebo reference="drop_ir_rr">
-   <sensor type="ray" name="TeraRanger">
-      <pose>0 0 0 0 0 0</pose>
-      <visualize>true</visualize>
-      <update_rate>50</update_rate>
-      <ray>
-         <scan>
-            <horizontal>
-               <samples>10</samples>
-               <resolution>1</resolution>
-               <min_angle>-0.14835</min_angle>
-               <max_angle>0.14835</max_angle>
-            </horizontal>
-            <vertical>
-               <samples>10</samples>
-               <resolution>1</resolution>
-               <min_angle>-0.14835</min_angle>
-               <max_angle>0.14835</max_angle>
-            </vertical>
-         </scan>
-         <range>
-            <min>0.01</min>
-            <max>2</max>
-            <resolution>0.02</resolution>
-         </range>
-      </ray>
-      <plugin filename="libgazebo_ros_range.so" name="gazebo_ros_range">
-         <gaussianNoise>0.005</gaussianNoise>
-         <alwaysOn>true</alwaysOn>
-         <updateRate>50</updateRate>
-         <topicName>drop_sensor_rr</topicName>
-         <frameName>drop_ir_rr</frameName>
-         <radiation>INFRARED</radiation>
-         <fov>0.2967</fov>
-      </plugin>
-   </sensor>
-   </gazebo>
+  </xacro:drop_sensor>
 </robot>
