Commit message: cozmo mesh package reference fixed

File: urdf/cozmo.xacro (robot description, xacro)
@@ -15,10 +15,10 @@
       <geometry>
         <!-- TODO: check why this collada file won't load into gazebo -->
-        <mesh filename="package://cozmo_description/meshes/body3.dae"  />
+        <mesh filename="package://anki_description/meshes/body3.dae"  />
       </geometry>
     </visual>
     <collision>
       <geometry>
-        <mesh filename="package://cozmo_description/meshes/body3.dae"  />
+        <mesh filename="package://anki_description/meshes/body3.dae"  />
       </geometry>
     </collision>
@@ -36,10 +36,10 @@
     <visual>
       <geometry>
-        <mesh filename="package://cozmo_description/meshes/cozmo_head.dae" />
+        <mesh filename="package://anki_description/meshes/cozmo_head.dae" />
       </geometry>
     </visual>
     <collision>
       <geometry>
-        <mesh filename="package://cozmo_description/meshes/cozmo_head.dae"/>
+        <mesh filename="package://anki_description/meshes/cozmo_head.dae"/>
       </geometry>
     </collision>
@@ -57,10 +57,10 @@
     <visual>
       <geometry>
-        <mesh filename="package://cozmo_description/meshes/cozmo_lift.dae"/>
+        <mesh filename="package://anki_description/meshes/cozmo_lift.dae"/>
       </geometry>
     </visual>
     <collision>
       <geometry>
-        <mesh filename="package://cozmo_description/meshes/cozmo_lift.dae"/>
+        <mesh filename="package://anki_description/meshes/cozmo_lift.dae"/>
       </geometry>
     </collision>
