Commit message: refinements

File: urdf/base.xacro (robot description, xacro)
@@ -4,4 +4,5 @@
     <link name="${link_name}">
       <visual>
+        <material name="black"/>
         <origin rpy="0 0 0" xyz="0 0 0"/>
         <geometry>
@@ -10,4 +11,5 @@
       </visual>
       <collision>
+        <material name="black"/>
         <origin rpy="0 0 0" xyz="0 0 0"/>
         <geometry>
@@ -33,4 +35,11 @@
         </actuator>
     </transmission>
+    <!-- <gazebo reference="${link_name}">
+      <selfCollide>true</selfCollide>
+      <mu1 value="200.0"/>
+      <mu2 value="100.0"/>
+      <kp value="10000000.0"/>
+      <kd value="1.0"/>
+    </gazebo> -->
   </xacro:macro>
 <xacro:wheel link_name="front_left_wheel" radius="0.01314">

File: urdf/cozmo.xacro (robot description, xacro)
@@ -5,5 +5,5 @@
   <link name="base_footprint"/>
   <joint name="base_footprint_joint" type="fixed">
-    <origin rpy="0 0 0" xyz="0 0 0.026"/>
+    <origin rpy="0 0 0" xyz="0 0 0.027"/>
     <parent link="base_footprint"/>
     <child link="base_link"/>
@@ -72,4 +72,4 @@
   <xacro:include filename="$(find anki_description)/urdf/cozmo_drop.xacro"/>
   <xacro:include filename="$(find anki_description)/urdf/imu.xacro"/>
-  <xacro:imu name="cozmo"/>
+  <xacro:imu ankirobot="cozmo"/>
 </robot>

File: urdf/cozmo_cam.xacro (robot description, xacro)
@@ -37,5 +37,5 @@
           <updateRate>10.0</updateRate>
           <cameraName>cozmo_camera</cameraName>
-          <imageTopicName>/cozmo/image</imageTopicName>
+          <imageTopicName>/cozmo/camera</imageTopicName>
           <cameraInfoTopicName>/cozmo/camera_info</cameraInfoTopicName>
           <frameName>camera_link</frameName>

File: urdf/cozmo_drop.xacro (robot description, xacro)
@@ -14,39 +14,39 @@
   </joint>
   <gazebo reference="drop_ir">
-  <sensor type="ray" name="ranger">
-    <pose>0 0 0 0 0 0</pose>
-    <visualize>true</visualize>
-    <update_rate>50</update_rate>
-    <ray>
-       <scan>
-          <horizontal>
-             <samples>10</samples>
-             <resolution>1</resolution>
-             <min_angle>-0.14835</min_angle>
-             <max_angle>0.14835</max_angle>
-          </horizontal>
-          <vertical>
-             <samples>10</samples>
-             <resolution>1</resolution>
-             <min_angle>-0.14835</min_angle>
-             <max_angle>0.14835</max_angle>
-          </vertical>
-       </scan>
-       <range>
-          <min>0.001</min>
-          <max>0.02</max>
-          <resolution>0.02</resolution>
-       </range>
-    </ray>
-    <plugin filename="libgazebo_ros_range.so" name="gazebo_ros_range">
-       <gaussianNoise>0.005</gaussianNoise>
-       <alwaysOn>true</alwaysOn>
-       <updateRate>50</updateRate>
-       <topicName>/cozmo/drop_sensor</topicName>
-       <frameName>drop_ir</frameName>
-       <radiation>INFRARED</radiation>
-       <fov>0.2967</fov>
-    </plugin>
-  </sensor>
+    <sensor type="ray" name="ranger">
+      <pose>0 0 0 0 0 0</pose>
+      <visualize>true</visualize>
+      <update_rate>50</update_rate>
+      <ray>
+         <scan>
+            <horizontal>
+               <samples>10</samples>
+               <resolution>1</resolution>
+               <min_angle>-0.14835</min_angle>
+               <max_angle>0.14835</max_angle>
+            </horizontal>
+            <vertical>
+               <samples>10</samples>
+               <resolution>1</resolution>
+               <min_angle>-0.14835</min_angle>
+               <max_angle>0.14835</max_angle>
+            </vertical>
+         </scan>
+         <range>
+            <min>0.001</min>
+            <max>0.02</max>
+            <resolution>0.02</resolution>
+         </range>
+      </ray>
+      <plugin filename="libgazebo_ros_range.so" name="gazebo_ros_range">
+         <gaussianNoise>0.005</gaussianNoise>
+         <alwaysOn>true</alwaysOn>
+         <updateRate>50</updateRate>
+         <topicName>/cozmo/drop_sensor</topicName>
+         <frameName>drop_ir</frameName>
+         <radiation>INFRARED</radiation>
+         <fov>0.2967</fov>
+      </plugin>
+    </sensor>
   </gazebo>
 </robot>

File: urdf/joints.xacro (robot description, xacro)
@@ -6,5 +6,5 @@
     <origin xyz="0.0174507 0 0.022003"/>
     <limit lower="-0.52" upper="0.17" effort="100" velocity="10"/>
-    <!-- Dampnening breaks the model (?), keep it 0.0 -->
+    <!-- Damping breaks the model (?), keep it 0.0 -->
     <dynamics damping="0.0" friction="0.1"/>
     <axis xyz="0 1 0"/>
@@ -22,9 +22,10 @@
       <type>transmission_interface/SimpleTransmission</type>
       <joint name="base_to_head">
-        <hardwareInterface>hardware_interface/EffortJointInterface</hardwareInterface>
+        <hardwareInterface>hardware_interface/PositionJointInterface</hardwareInterface>
       </joint>
       <actuator name="base_to_headMotor">
-        <hardwareInterface>hardware_interface/EffortJointInterface</hardwareInterface>
+        <hardwareInterface>hardware_interface/PositionJointInterface</hardwareInterface>
         <mechanicalReduction>1</mechanicalReduction>
+        <motorTorqueConstant>1</motorTorqueConstant>
       </actuator>
   </transmission>
@@ -32,9 +33,10 @@
       <type>transmission_interface/SimpleTransmission</type>
       <joint name="base_to_lift">
-        <hardwareInterface>hardware_interface/EffortJointInterface</hardwareInterface>
+        <hardwareInterface>hardware_interface/PositionJointInterface</hardwareInterface>
       </joint>
       <actuator name="base_to_liftMotor">
-        <hardwareInterface>hardware_interface/EffortJointInterface</hardwareInterface>
+        <hardwareInterface>hardware_interface/PositionJointInterface</hardwareInterface>
         <mechanicalReduction>1</mechanicalReduction>
+        <motorTorqueConstant>1</motorTorqueConstant>
       </actuator>
   </transmission>

File: urdf/laser.xacro (robot description, xacro)
@@ -1,20 +1,10 @@
 <?xml version="1.0"?>
 <robot xmlns:xacro="http://www.ros.org/wiki/xacro">
-  <link name="tof_link">
-      <visual>
-          <geometry>
-              <box size="0.001 0.001 0.001"/>
-          </geometry>
-      </visual>
-      <collision>
-          <geometry>
-              <box size="0.001 0.001 0.001"/>
-          </geometry>
-      </collision>
-  </link>
+  <xacro:property name="field_of_view" value="0.02"/>
+  <link name="tof_link"/>
   <joint name="tof_joint" type="fixed">
       <parent link="base_link"/>
       <child link="tof_link"/>
-      <origin rpy="0 0 0" xyz="0.022 0 0.03"/>
+      <origin rpy="0 0 0" xyz="0.042 0 -0.005"/>
   </joint>
   <gazebo reference="tof_link">
@@ -28,17 +18,17 @@
                       <samples>4</samples>
                       <resolution>1</resolution>
-                      <min_angle>-0.001</min_angle>
-                      <max_angle>0.001</max_angle>
+                      <min_angle>${-field_of_view/2}</min_angle>
+                      <max_angle>${field_of_view/2}</max_angle>
                   </horizontal>
                   <vertical>
                       <samples>4</samples>
                       <resolution>1</resolution>
-                      <min_angle>-0.001</min_angle>
-                      <max_angle>0.001</max_angle>
+                      <min_angle>${-field_of_view/2}</min_angle>
+                      <max_angle>${field_of_view/2}</max_angle>
                   </vertical>
               </scan>
               <range>
                   <min>0.0</min>
-                  <max>0.3</max>
+                  <max>0.4</max>
                   <resolution>0.01</resolution>
               </range>
@@ -46,5 +36,5 @@
                 <type>gaussian</type>
                 <mean>0.01</mean>
-                <stddev>0.04</stddev>
+                <stddev>0.01</stddev>
               </noise>
           </ray>
@@ -55,5 +45,5 @@
               <radiation>INFRARED</radiation>
               <updateRate>20</updateRate>
-              <fov>0.2617993878</fov>
+              <fov>${field_of_view}</fov>
           </plugin>
       </sensor>

File: urdf/vector.xacro (robot description, xacro)
@@ -5,5 +5,5 @@
   <link name="base_footprint"/>
   <joint name="base_footprint_joint" type="fixed">
-    <origin rpy="0 0 0" xyz="0 0 0.026"/>
+    <origin rpy="0 0 0" xyz="0 0 0.027"/>
     <parent link="base_footprint"/>
     <child link="base_link"/>

File: urdf/vector_cam.xacro (robot description, xacro)
@@ -31,5 +31,5 @@
         <updateRate>10.0</updateRate>
         <cameraName>camera</cameraName>
-        <imageTopicName>/vector/image</imageTopicName>
+        <imageTopicName>/vector/camera</imageTopicName>
         <cameraInfoTopicName>/vector/camera_info</cameraInfoTopicName>
         <frameName>camera_link</frameName>

Commit message: inertia fix

File: urdf/base.xacro (robot description, xacro)
@@ -17,6 +17,16 @@
         </geometry>
       </collision>
-      <xacro:cylinder_inertial mass="0.005" radius="${radius}" length="0.01167"/>
+      <inertial>
+        <origin rpy="0 0 0" xyz="0 0 0"/>
+        <geometry>
+          <cylinder radius="${radius}" length="0.0116739"/>
+        </geometry>
+        <mass value="0.01"/>
+        <xacro:cylinder_inertia m="0.01" r="${radius}" h="0.01167"/>
+      </inertial>
     </link>
+    <gazebo reference="${link_name}">
+      <material>Gazebo/Grey</material>
+    </gazebo>
     <joint name="${link_name}_joint" type="continuous">
         <parent link="base_link"/>
@@ -35,11 +45,11 @@
         </actuator>
     </transmission>
-    <!-- <gazebo reference="${link_name}">
-      <selfCollide>true</selfCollide>
-      <mu1 value="200.0"/>
+    <gazebo reference="${link_name}">
+      <selfCollide>True</selfCollide>
+      <!-- <mu1 value="200.0"/>
       <mu2 value="100.0"/>
       <kp value="10000000.0"/>
-      <kd value="1.0"/>
-    </gazebo> -->
+      <kd value="1.0"/> -->
+    </gazebo>
   </xacro:macro>
 <xacro:wheel link_name="front_left_wheel" radius="0.01314">
@@ -90,5 +100,5 @@
         <wheelDiameter>0.026281</wheelDiameter>
         <robotBaseFrame>base_footprint</robotBaseFrame>
-        <torque>0.1</torque>
+        <torque>1.0</torque>
         <commandTopic>cmd_vel</commandTopic>
         <odometryTopic>odom</odometryTopic>

File: urdf/cozmo.xacro (robot description, xacro)
@@ -1,4 +1,4 @@
 <?xml version="1.0"?>
-<robot name="cozmo" xmlns:xacro="http://www.ros.org/wiki/xacro">
+<robot name="robot" xmlns:xacro="http://www.ros.org/wiki/xacro">
   <!-- Inertia util -->
   <xacro:include filename="$(find anki_description)/urdf/inertia.xacro"/>
@@ -11,5 +11,4 @@
   <!-- Body -->
   <link name="base_link">
-    <xacro:box_inertial mass="0.06" x="0.073" y="0.043" z="0.061" />
     <visual>
       <geometry>
@@ -24,4 +23,8 @@
     </collision>
   </link>
+  <inertial>
+    <mass value="0.06"/>
+    <xacro:box_inertia m="0.06" x="0.073" y="0.043" z="0.061" />
+  </inertial>
   <gazebo reference="base_link">
       <selfCollide>true</selfCollide>
@@ -33,5 +36,4 @@
   <!-- Head -->
   <link name="head">
-    <xacro:box_inertial mass="0.01" x="0.036" y="0.038" z="0.041" />
     <visual>
       <geometry>
@@ -44,4 +46,8 @@
       </geometry>
     </collision>
+    <inertial>
+      <mass value="0.01"/>
+      <xacro:box_inertia m="0.01" x="0.036" y="0.038" z="0.041" />
+    </inertial>
   </link>
   <gazebo reference="head">
@@ -54,5 +60,5 @@
   <!-- lifter -->
   <link name="full_lift">
-    <xacro:box_inertial mass="0.01" x="0.081" y="0.058" z="0.050"/>
+    <xacro:box_inertia m="0.01" x="0.081" y="0.058" z="0.050"/>
     <visual>
       <geometry>

File: urdf/inertia.xacro (robot description, xacro)
@@ -1,23 +1,18 @@
 <?xml version="1.0"?>
 <robot xmlns:xacro="http://www.ros.org/wiki/xacro">
-  <xacro:macro name="cylinder_inertial" params="radius length mass">
-    <inertial>
-      <mass value="${mass}" />
-      <inertia ixx="${0.0833333 * mass * (3 * radius * radius + length * length)}" ixy="0.0" ixz="0.0"
-        izz="${0.0833333 * mass * (3 * radius * radius + length * length)}" iyz="0.0"
-        iyy="${0.5 * mass * radius * radius}" />
-    </inertial>
-  </xacro:macro>
-  <xacro:macro name="box_inertial" params="mass x y z">
-    <inertial>
-      <mass value="${mass}" />
-      <inertia  ixx="${mass*(y*y+z*z)/12}" ixy = "0" ixz = "0" iyy="${mass*(x*x+z*z)/12}" iyz = "0" izz="${mass*(x*x+z*z)/12}" />
-    </inertial>
-  </xacro:macro>
-    <xacro:macro name="box_inertial_default" params="mass">
-    <inertial>
-      <mass value="${mass}" />
-      <inertia  ixx="0.000001" ixy = "0" ixz = "0" iyy="0.000001" iyz = "0" izz="0.0000001" />
-    </inertial>
-  </xacro:macro>
+  <macro name="cylinder_inertia" params="m r h">
+        <inertia    ixx="${m*(3*r*r+h*h)/12}" ixy = "0" ixz = "0"
+                    iyy="${m*(3*r*r+h*h)/12}" iyz = "0"
+                    izz="${m*r*r/2}" />
+  </macro>
+  <macro name="box_inertia" params="m x y z">
+          <inertia  ixx="${m*(y*y+z*z)/12}" ixy = "0" ixz = "0"
+                    iyy="${m*(x*x+z*z)/12}" iyz = "0"
+                    izz="${m*(x*x+z*z)/12}" />
+  </macro>
+  <macro name="sphere_inertia" params="m r">
+          <inertia  ixx="${2*m*r*r/5}" ixy = "0" ixz = "0"
+                    iyy="${2*m*r*r/5}" iyz = "0"
+                    izz="${2*m*r*r/5}" />
+  </macro>
 </robot>

File: urdf/joints.xacro (robot description, xacro)
@@ -14,5 +14,5 @@
     <child link="full_lift"/>
     <origin xyz="-0.005 0 0.013"/>
-    <limit lower="-0.8" upper="0" effort="5" velocity="10"/>
+    <limit lower="-0.8" upper="0" effort="10" velocity="10"/>
     <dynamics damping="0.0" friction="0.1"/>
     <axis xyz="0 1 0"/>

File: urdf/vector.xacro (robot description, xacro)
@@ -11,5 +11,4 @@
   <!-- Body -->
   <link name="base_link">
-    <xacro:box_inertial mass="0.06" x="0.073" y="0.043" z="0.061" />
     <visual>
       <geometry>
@@ -18,8 +17,18 @@
     </visual>
     <collision>
+      <origin rpy="0 0 0" xyz="0.0075 0.0 -0.01"/>
       <geometry>
-        <mesh filename="package://anki_description/meshes/vector_body.dae"  />
+        <box size="0.07 0.03 0.01"/>
+        <!-- <mesh filename="package://anki_description/meshes/vector_body.dae"  /> -->
       </geometry>
     </collision>
+    <inertial>
+      <origin rpy="0 0 0" xyz="0.0075 0.0 -0.01"/>
+      <geometry>
+        <box size="0.073 0.043 0.061"/>
+      </geometry>
+      <mass value="0.16"/>
+      <xacro:box_inertia m="0.16" x="0.073" y="0.043" z="0.061" />
+    </inertial>
   </link>
   <gazebo reference="base_link">
@@ -32,5 +41,4 @@
   <!-- Head -->
   <link name="head">
-    <xacro:box_inertial mass="0.01" x="0.036" y="0.038" z="0.041" />
     <visual>
       <geometry>
@@ -40,18 +48,23 @@
     <collision>
       <geometry>
-        <mesh filename="package://anki_description/meshes/vector_head.dae"/>
+        <sphere radius="0.02"/>
       </geometry>
     </collision>
+    <inertial>
+      <geometry>
+        <sphere radius="0.02"/>
+      </geometry>
+      <mass value="0.03"/>
+      <xacro:sphere_inertia m="0.03" r="0.02" />
+    </inertial>
   </link>
   <gazebo reference="head">
-      <kp>1000000000.0</kp>
-      <kd>1000000000.0</kd>
-      <mu1>10.0</mu1>
-      <mu2>10.0</mu2>
-      <self_collide>0</self_collide>
+    <mu1 value="200.0"/>
+    <mu2 value="100.0"/>
+    <kp value="10000000.0"/>
+    <kd value="1.0"/>
   </gazebo>
   <!-- lifter -->
   <link name="full_lift">
-    <xacro:box_inertial mass="0.01" x="0.081" y="0.058" z="0.050"/>
     <visual>
       <geometry>
@@ -60,9 +73,24 @@
     </visual>
     <collision>
+      <origin rpy="0 0 0" xyz="0.062 0.0 -0.015"/>
       <geometry>
-        <mesh filename="package://anki_description/meshes/vector_lift.dae"/>
+        <box size="0.0075 0.05 0.025"/>
       </geometry>
     </collision>
+    <inertial>
+      <origin rpy="0 0 0" xyz="0.062 0.0 -0.015"/>
+      <geometry>
+        <box size="0.0075 0.05 0.025"/>
+      </geometry>
+      <mass value="0.05"/>
+      <xacro:box_inertia m="0.05" x="0.0075" y="0.05" z="0.025"/>
+    </inertial>
   </link>
+  <gazebo reference="full_lift">
+    <mu1 value="200.0"/>
+    <mu2 value="100.0"/>
+    <kp value="10000000.0"/>
+    <kd value="1.0"/>
+  </gazebo>
   <!-- components -->
   <xacro:include filename="$(find anki_description)/urdf/joints.xacro"/>
