Commit message: xacro:macro

File: urdf/inertia.xacro (robot description, xacro)
@@ -1,18 +1,18 @@
 <?xml version="1.0"?>
 <robot xmlns:xacro="http://www.ros.org/wiki/xacro">
-  <macro name="cylinder_inertia" params="m r h">
+  <xacro:macro name="cylinder_inertia" params="m r h">
         <inertia    ixx="${m*(3*r*r+h*h)/12}" ixy = "0" ixz = "0"
                     iyy="${m*(3*r*r+h*h)/12}" iyz = "0"
                     izz="${m*r*r/2}" />
-  </macro>
-  <macro name="box_inertia" params="m x y z">
+  </xacro:macro>
+  <xacro:macro name="box_inertia" params="m x y z">
           <inertia  ixx="${m*(y*y+z*z)/12}" ixy = "0" ixz = "0"
                     iyy="${m*(x*x+z*z)/12}" iyz = "0"
                     izz="${m*(x*x+z*z)/12}" />
-  </macro>
-  <macro name="sphere_inertia" params="m r">
+  </xacro:macro>
+  <xacro:macro name="sphere_inertia" params="m r">
           <inertia  ixx="${2*m*r*r/5}" ixy = "0" ixz = "0"
                     iyy="${2*m*r*r/5}" iyz = "0"
                     izz="${2*m*r*r/5}" />
-  </macro>
+  </xacro:macro>
 </robot>
